Commit message: Fixed package name error in urdf macros

File: cyton_gamma_300.urdf.xacro (robot description, xacro)
@@ -1,5 +1,5 @@
 <?xml version="1.0"?>
 <robot xmlns:xacro="http://www.ros.org/wiki/xacro" name="cyton_gamma_300">
-  <xacro:include filename="$(find cyton_gamma_300)/cyton_gamma_300_macros.urdf.xacro" />
+  <xacro:include filename="$(find cyton_gamma_300_description)/cyton_gamma_300_macros.urdf.xacro" />
   <xacro:base_footprint prefix="" />
   <xacro:cyton_gamma_300 prefix="" virtual_ee="true" />

File: cyton_gamma_300_macros.urdf.xacro (robot description, xacro)
@@ -26,5 +26,5 @@
                 <origin xyz="0 0 0" rpy="0 0 0"/>
                 <geometry>
-                    <mesh filename="package://cyton_gamma_300/meshes/gamma_base.dae"/>
+                    <mesh filename="package://cyton_gamma_300_description/meshes/gamma_base.dae"/>
                 </geometry>
             </visual>
@@ -48,5 +48,5 @@
                 <origin xyz="0 0 0" rpy="0 0 0"/>
                 <geometry>
-                    <mesh filename="package://cyton_gamma_300/meshes/Shoulder_Roll.dae"/>
+                    <mesh filename="package://cyton_gamma_300_description/meshes/Shoulder_Roll.dae"/>
                 </geometry>
             </visual>
@@ -70,5 +70,5 @@
                 <origin xyz="0 0 0" rpy="0 1.5708 0" />
                 <geometry>
-                    <mesh filename="package://cyton_gamma_300/meshes/Shoulder_Pitch.dae"/>
+                    <mesh filename="package://cyton_gamma_300_description/meshes/Shoulder_Pitch.dae"/>
                 </geometry>
             </visual>
@@ -92,5 +92,5 @@
                 <origin xyz="0 0 0.0" rpy="0 0 0" />
                 <geometry>
-                    <mesh filename="package://cyton_gamma_300/meshes/Elbow_Roll.dae"/>
+                    <mesh filename="package://cyton_gamma_300_description/meshes/Elbow_Roll.dae"/>
                 </geometry>
             </visual>
@@ -115,5 +115,5 @@
                 <origin xyz="0 0 0" rpy="1.5708 0 0.7854" />
                 <geometry>
-                    <mesh filename="package://cyton_gamma_300/meshes/Elbow_Pitch.dae"/>
+                    <mesh filename="package://cyton_gamma_300_description/meshes/Elbow_Pitch.dae"/>
                 </geometry>
             </visual>
@@ -137,5 +137,5 @@
                 <origin xyz="0 0 0" rpy="1.5708 0 2.3562" />
                 <geometry>
-                    <mesh filename="package://cyton_gamma_300/meshes/Elbow_Yaw.dae"/>
+                    <mesh filename="package://cyton_gamma_300_description/meshes/Elbow_Yaw.dae"/>
                 </geometry>
             </visual>
@@ -159,5 +159,5 @@
                 <origin xyz="0 0 0" rpy="1.5708 0 0.7854" />
                 <geometry>
-                    <mesh filename="package://cyton_gamma_300/meshes/Wrist_Pitch.dae"/>
+                    <mesh filename="package://cyton_gamma_300_description/meshes/Wrist_Pitch.dae"/>
                 </geometry>
             </visual>
@@ -181,5 +181,5 @@
                 <origin xyz="0 0 0" rpy="3.1416 0 -2.3562" />
                 <geometry>
-                    <mesh filename="package://cyton_gamma_300/meshes/Wrist_Roll.dae"/>
+                    <mesh filename="package://cyton_gamma_300_description/meshes/Wrist_Roll.dae"/>
                 </geometry>
             </visual>
@@ -203,5 +203,5 @@
                 <origin xyz="0 0 0" rpy="0 0 0" />
                 <geometry>
-                    <mesh filename="package://cyton_gamma_300/meshes/Gripper_Finger1.dae"/>
+                    <mesh filename="package://cyton_gamma_300_description/meshes/Gripper_Finger1.dae"/>
                 </geometry>
             </visual>
@@ -226,5 +226,5 @@
                 <origin xyz="0 0 0" rpy="0 0 0" />
                 <geometry>
-                    <mesh filename="package://cyton_gamma_300/meshes/Gripper_Finger2.dae"/>
+                    <mesh filename="package://cyton_gamma_300_description/meshes/Gripper_Finger2.dae"/>
                 </geometry>
             </visual>
