Commit message: Set up URDF macros properly

File: cyton_gamma_300_macros.urdf.xacro (robot description, xacro)
@@ -40,5 +40,5 @@
             <parent link="${prefix}base_link" />
             <child link="${prefix}shoulder_roll" />
-            <origin xyz="0 0 0.05315" rpy="1.5708 0 0" />
+            <origin xyz="0 0 0.05315" rpy="0 0 1.2" />
             <limit lower="-2.618" upper="2.618" effort="100.0" velocity="1.0" />
             <axis xyz="0 0 1" />
@@ -46,5 +46,5 @@
         <link name="${prefix}shoulder_roll">
             <visual>
-                <origin xyz="0 0 0" rpy="0 0 0"/>
+                <origin xyz="0 0 0" rpy="1.5708 0 3.14159"/>
                 <geometry>
                     <mesh filename="package://cyton_gamma_300_description/meshes/Shoulder_Roll.dae"/>
@@ -62,5 +62,5 @@
             <parent link="${prefix}shoulder_roll" />
             <child link="${prefix}shoulder_pitch" />
-            <origin xyz="0.028 0 0.063" rpy="0 0 0" />
+            <origin xyz="0 0 0.063" rpy="1.2 0 0" />
             <limit lower="-1.8326" upper="1.8326" effort="100.0" velocity="1.0" />
             <axis xyz="1 0 0" />
@@ -68,5 +68,5 @@
         <link name="${prefix}shoulder_pitch">
             <visual>
-                <origin xyz="0 0 0" rpy="0 1.5708 0" />
+                <origin xyz="0.028 0 0" rpy="0 1.5708 0" />
                 <geometry>
                     <mesh filename="package://cyton_gamma_300_description/meshes/Shoulder_Pitch.dae"/>
@@ -84,11 +84,11 @@
             <parent link="${prefix}shoulder_pitch" />
             <child link="${prefix}elbow_roll" />
-            <origin xyz="-0.028 0 0.089" rpy="0 0 0" />
-            <limit lower="-1.8326" upper="1.8326" effort="100.0" velocity="1.0" />
-            <axis xyz="0 -1 0" />
+            <origin xyz="0 0 0.089" rpy="0 0 1.2" />
+            <limit lower="-1.8326" upper="1.8326" effort="100.0" velocity="1.0" />
+            <axis xyz="0 0 1" />
         </joint>
         <link name="${prefix}elbow_roll">
             <visual>
-                <origin xyz="0 0 0.0" rpy="0 0 0" />
+                <origin xyz="0 0 0" rpy="0 0 3.92699" />
                 <geometry>
                     <mesh filename="package://cyton_gamma_300_description/meshes/Elbow_Roll.dae"/>
@@ -102,9 +102,9 @@
             </collision>
         </link>
-        <!-- Third motor located here -->
+        <!-- Fourth motor located here -->
         <joint name="${prefix}elbow_pitch_joint" type="revolute">
             <parent link="${prefix}elbow_roll" />
             <child link="${prefix}elbow_pitch" />
-            <origin xyz="0.018 -0.018 0.052" rpy="0 0 0" />
+            <origin xyz="0 0 0.052" rpy="1.2 0 0" />
             <limit lower="-1.8326" upper="1.8326" effort="100.0" velocity="1.0" />
             <axis xyz="1 0 0" />
@@ -113,5 +113,5 @@
             <visual>
                 <!-- Not sure if this is the correct orientation. -->
-                <origin xyz="0 0 0" rpy="1.5708 0 0.7854" />
+                <origin xyz="0.027 0 0" rpy="1.5708 0 1.5708" />
                 <geometry>
                     <mesh filename="package://cyton_gamma_300_description/meshes/Elbow_Pitch.dae"/>
@@ -125,9 +125,9 @@
             </collision>
         </link>
-        <!-- Fourth motor located here -->
+        <!-- Fifth motor located here -->
         <joint name="${prefix}elbow_yaw_joint" type="revolute">
             <parent link="${prefix}elbow_pitch" />
             <child link="${prefix}elbow_yaw" />
-            <origin xyz="-0.018 0.018 0.072" rpy="0 0 0" />
+            <origin xyz="0 0 0.072" rpy="0 -1.2 0" />
             <limit lower="-1.8326" upper="1.8326" effort="100.0" velocity="1.0" />
             <axis xyz="0 -1 0" />
@@ -135,5 +135,5 @@
         <link name="${prefix}elbow_yaw">
             <visual>
-                <origin xyz="0 0 0" rpy="1.5708 0 2.3562" />
+                <origin xyz="0 0 0" rpy="1.5708 0 0" />
                 <geometry>
                     <mesh filename="package://cyton_gamma_300_description/meshes/Elbow_Yaw.dae"/>
@@ -147,9 +147,9 @@
             </collision>
         </link>
-        <!-- Fifth motor located here -->
+        <!-- Sixth motor located here -->
         <joint name="${prefix}wrist_pitch_joint" type="revolute">
             <parent link="${prefix}elbow_yaw" />
             <child link="${prefix}wrist_pitch" />
-            <origin xyz="0.018 -0.018 0.0718" rpy="0 0 0" />
+            <origin xyz="0 0 0.0718" rpy="1.2 0 0" />
             <limit lower="-1.8326" upper="1.8326" effort="100.0" velocity="1.0" />
             <axis xyz="1 0 0" />
@@ -157,5 +157,5 @@
         <link name="${prefix}wrist_pitch">
             <visual>
-                <origin xyz="0 0 0" rpy="1.5708 0 0.7854" />
+                <origin xyz="0.027 0 0" rpy="1.5708 0 1.5708" />
                 <geometry>
                     <mesh filename="package://cyton_gamma_300_description/meshes/Wrist_Pitch.dae"/>
@@ -169,9 +169,9 @@
             </collision>
         </link>
-        <!-- Sixth motor located here -->
+        <!-- Seventh motor located here -->
         <joint name="${prefix}wrist_roll_joint" type="revolute">
             <parent link="${prefix}wrist_pitch" />
             <child link="${prefix}wrist_roll" />
-            <origin xyz="-0.018 0.018 0.051425" rpy="0 0 0" />
+            <origin xyz="0 0 0.051425" rpy="0 0 1.2" />
             <limit lower="-2.61799" upper="2.61799" effort="100.0" velocity="1.0" />
             <axis xyz="0 0 1" />
@@ -179,5 +179,5 @@
         <link name="${prefix}wrist_roll">
             <visual>
-                <origin xyz="0 0 0" rpy="3.1416 0 -2.3562" />
+                <origin xyz="0 0 0" rpy="0 3.14159 1.5708" />
                 <geometry>
                     <mesh filename="package://cyton_gamma_300_description/meshes/Wrist_Roll.dae"/>
@@ -191,5 +191,5 @@
             </collision>
         </link>
-        <!-- Seventh motor located here -->
+        <!-- Eigth motor located here -->
         <joint name="${prefix}gripper_joint" type="prismatic">
             <parent link="${prefix}wrist_roll" />
