Commit message: xacro file modified to support different transmission types, gazebo simulation package added

File: cyton_gamma_300_description/urdf/cyton_gamma_300.urdf.xacro (robot description, xacro)
@@ -5,4 +5,8 @@
 	<!-- Import Rviz colors -->
 	<xacro:include filename="$(find cyton_gamma_300_description)/urdf/materials.xacro" />
+	<!-- ########################################### -->
+	<!-- #######! PROPERTIES !###################### -->
+	<!-- ########################################### -->
+	<xacro:property name="transmission" value="$(arg transmission)" />
 	<!-- Used for fixing robot to Gazebo 'base_link' -->
 	<link name="world">
@@ -440,12 +444,12 @@
     </xacro:macro>
   <xacro:cyton_gamma_300 virtual_ee="true" />
-  <xacro:macro name="include_transmission" params="transmission_type">
-	<xacro:if value="${transmission_type == 'position'}">
+  <xacro:macro name="include_transmission" >
+	<xacro:if value="${transmission == 'position'}">
 		<xacro:include filename="$(find cyton_gamma_300_description)/urdf/transmissions_positionjointinterface.xml" />
 	</xacro:if>
-	<xacro:if value="${transmission_type == 'effort'}">
+	<xacro:if value="${transmission == 'effort'}">
 	   <xacro:include filename="$(find cyton_gamma_300_description)/urdf/transmissions_effortjointinterface.xml" />
 	</xacro:if>
   </xacro:macro>
-  <xacro:include_transmission transmission_type="position" />
+  <xacro:include_transmission  />
 </robot>

Commit message: gazebo moveit simulation includes robot

File: cyton_gamma_300_description/urdf/cyton_gamma_300.urdf.xacro (robot description, xacro)
@@ -93,5 +93,5 @@
             <parent link="shoulder_roll" />
             <child link="shoulder_pitch" />
-            <origin xyz="0 0 0.063" rpy="0.0 0 0" />
+            <origin xyz="0 0 0.063" rpy="1.2 0 0" />
             <limit lower="-1.8326" upper="1.8326" effort="100.0" velocity="1.0" />
             <axis xyz="1 0 0" />

Commit message: refactoring urdf for initial arm pose in simulation

File: cyton_gamma_300_description/urdf/cyton_gamma_300.urdf.xacro (robot description, xacro)
@@ -9,4 +9,37 @@
 	<!-- ########################################### -->
 	<xacro:property name="transmission" value="$(arg transmission)" />
+	<xacro:property name="shoulder_roll_joint_init_xyz" 		value="0 0 0.05315" />
+	<xacro:property name="shoulder_roll_joint_init_rpy" 		value="0 0 1.2" />
+	<xacro:property name="shoulder_pitch_joint_init_xyz" 		value="0 0 0.063" />
+	<xacro:property name="shoulder_pitch_joint_init_rpy" 		value="1.2 0 0" />
+	<xacro:property name="elbow_roll_joint_init_xyz" 			value="0 0 0.089" />
+	<xacro:property name="elbow_roll_joint_init_rpy" 			value="0 0 1.2" />
+	<xacro:property name="elbow_pitch_joint_init_xyz" 			value="0 0 0.052" />
+	<xacro:property name="elbow_pitch_joint_init_rpy" 			value="1.2 0 0" />
+	<xacro:property name="elbow_yaw_joint_init_xyz" 			value="0 0 0.072" />
+	<xacro:property name="elbow_yaw_joint_init_rpy" 			value="0 -1.2 0" />
+	<xacro:property name="wrist_pitch_joint_init_xyz" 			value="0 0 0.0718" />
+	<xacro:property name="wrist_pitch_joint_init_rpy" 			value="1.2 0 0" />
+	<xacro:property name="wrist_roll_joint_init_xyz" 			value="0 0 0.051425" />
+	<xacro:property name="wrist_roll_joint_init_rpy" 			value="0 0 1.2" />
+	<xacro:property name="gripper_finger1_joint_init_xyz" 		value="-0.01331 0.00485 0.077225" />
+	<xacro:property name="gripper_finger1_joint_init_rpy" 		value="0 0 0" />
+	<xacro:property name="gripper_finger2_joint_init_xyz" 		value="0.0098 0.00485 0.077225" />
+	<xacro:property name="gripper_finger2_joint_init_rpy" 		value="0 0 0" />
+	<xacro:property name="virtual_endeffector_joint_init_xyz" 	value="-0.002316 0.0079 0.079425" />
+	<xacro:property name="virtual_endeffector_joint_init_rpy" 	value="0 0 0" />
+	<!-- ########################################### -->
+	<!-- #! SPECIFY INITIAL ARM POSITION   !######## -->
+	<!-- #! IN GAZEBO FROM THE LAUNCH FILE !######## -->
+	<!-- ########################################### -->
+	<xacro:if value="$(arg simulation)">
+	  <xacro:property name="shoulder_roll_joint_init_rpy" 		value="$(arg shoulder_roll_joint_init_rpy)" />
+	  <xacro:property name="shoulder_pitch_joint_init_rpy" 		value="$(arg shoulder_pitch_joint_init_rpy)" />
+	  <xacro:property name="elbow_roll_joint_init_rpy" 			value="$(arg elbow_roll_joint_init_rpy)" />
+	  <xacro:property name="elbow_pitch_joint_init_rpy" 		value="$(arg elbow_pitch_joint_init_rpy)" />
+	  <xacro:property name="elbow_yaw_joint_init_rpy" 			value="$(arg elbow_yaw_joint_init_rpy)" />
+	  <xacro:property name="wrist_pitch_joint_init_rpy" 		value="$(arg wrist_pitch_joint_init_rpy)" />
+	  <xacro:property name="wrist_roll_joint_init_rpy" 			value="$(arg wrist_roll_joint_init_rpy)" />
+	</xacro:if>
 	<!-- Used for fixing robot to Gazebo 'base_link' -->
 	<link name="world">
@@ -55,5 +88,5 @@
             <parent link="base_link" />
             <child link="shoulder_roll" />
-            <origin xyz="0 0 0.05315" rpy="0 0 1.2" />
+			<origin xyz="${shoulder_roll_joint_init_xyz}" rpy="${shoulder_roll_joint_init_rpy}" />
             <limit lower="-2.618" upper="2.618" effort="100.0" velocity="1.0" />
             <axis xyz="0 0 1" />
@@ -93,5 +126,5 @@
             <parent link="shoulder_roll" />
             <child link="shoulder_pitch" />
-            <origin xyz="0 0 0.063" rpy="1.2 0 0" />
+			<origin xyz="${shoulder_pitch_joint_init_xyz}" rpy="${shoulder_pitch_joint_init_rpy}" />
             <limit lower="-1.8326" upper="1.8326" effort="100.0" velocity="1.0" />
             <axis xyz="1 0 0" />
@@ -133,5 +166,5 @@
             <parent link="shoulder_pitch" />
             <child link="elbow_roll" />
-            <origin xyz="0 0 0.089" rpy="0 0 1.2" />
+			<origin xyz="${elbow_roll_joint_init_xyz}" rpy="${elbow_roll_joint_init_rpy}" />
             <limit lower="-1.8326" upper="1.8326" effort="100.0" velocity="1.0" />
             <axis xyz="0 0 1" />
@@ -173,5 +206,5 @@
             <parent link="elbow_roll" />
             <child link="elbow_pitch" />
-            <origin xyz="0 0 0.052" rpy="1.2 0 0" />
+			<origin xyz="${elbow_pitch_joint_init_xyz}" rpy="${elbow_pitch_joint_init_rpy}" />
             <limit lower="-1.8326" upper="1.8326" effort="100.0" velocity="1.0" />
             <axis xyz="1 0 0" />
@@ -215,5 +248,5 @@
             <parent link="elbow_pitch" />
             <child link="elbow_yaw" />
-            <origin xyz="0 0 0.072" rpy="0 -1.2 0" />
+			<origin xyz="${elbow_yaw_joint_init_xyz}" rpy="${elbow_yaw_joint_init_rpy}" />
             <limit lower="-1.8326" upper="1.8326" effort="100.0" velocity="1.0" />
             <axis xyz="0 -1 0" />
@@ -255,5 +288,5 @@
             <parent link="elbow_yaw" />
             <child link="wrist_pitch" />
-            <origin xyz="0 0 0.0718" rpy="1.2 0 0" />
+			<origin xyz="${wrist_pitch_joint_init_xyz}" rpy="${wrist_pitch_joint_init_rpy}" />
             <limit lower="-1.8326" upper="1.8326" effort="100.0" velocity="1.0" />
             <axis xyz="1 0 0" />
@@ -295,5 +328,5 @@
             <parent link="wrist_pitch" />
             <child link="wrist_roll" />
-            <origin xyz="0 0 0.051425" rpy="0 0 1.2" />
+			<origin xyz="${wrist_roll_joint_init_xyz}" rpy="${wrist_roll_joint_init_rpy}" />
             <limit lower="-2.61799" upper="2.61799" effort="100.0" velocity="1.0" />
             <axis xyz="0 0 1" />
@@ -335,5 +368,5 @@
             <parent link="wrist_roll" />
             <child link="gripper_finger1" />
-            <origin xyz="-0.01331 0.00485 0.077225" rpy="0 0 0" />
+			<origin xyz="${gripper_finger1_joint_init_xyz}" rpy="${gripper_finger1_joint_init_rpy}" />
             <limit lower="-0.008" upper="0.008" effort="100.0" velocity="1.0" />
             <axis xyz="1 0 0" />
@@ -375,5 +408,5 @@
             <parent link="wrist_roll" />
             <child link="gripper_finger2" />
-            <origin xyz="0.0098 0.00485 0.077225" rpy="0 0 0" />
+			<origin xyz="${gripper_finger2_joint_init_xyz}" rpy="${gripper_finger2_joint_init_rpy}" />
             <limit lower="-0.008" upper="0.008" effort="100.0" velocity="1.0" />
 			<mimic joint="gripper_finger1_joint" multiplier="-1"/>
@@ -415,5 +448,5 @@
                 <parent link="wrist_roll" />
                 <child link="virtual_endeffector" />
-                <origin xyz="-0.002316 0.0079 0.079425" rpy="0 0 0" />
+				<origin xyz="${virtual_endeffector_joint_init_xyz}" rpy="${virtual_endeffector_joint_init_rpy}" />
             </joint>
             <link name="virtual_endeffector">

Commit message: updating joint limits in xacro after measurement on the actual robot. removing now default `inorder` argument from the rviz lauch file

File: cyton_gamma_300_description/urdf/cyton_gamma_300.urdf.xacro (robot description, xacro)
@@ -89,5 +89,5 @@
             <child link="shoulder_roll" />
 			<origin xyz="${shoulder_roll_joint_init_xyz}" rpy="${shoulder_roll_joint_init_rpy}" />
-            <limit lower="-2.618" upper="2.618" effort="100.0" velocity="1.0" />
+            <limit lower="-3.9" upper="1.5" effort="100.0" velocity="1.0" />
             <axis xyz="0 0 1" />
         </joint>
@@ -127,5 +127,5 @@
             <child link="shoulder_pitch" />
 			<origin xyz="${shoulder_pitch_joint_init_xyz}" rpy="${shoulder_pitch_joint_init_rpy}" />
-            <limit lower="-1.8326" upper="1.8326" effort="100.0" velocity="1.0" />
+            <limit lower="-2.6" upper="0.2" effort="100.0" velocity="1.0" />
             <axis xyz="1 0 0" />
         </joint>
@@ -167,5 +167,5 @@
             <child link="elbow_roll" />
 			<origin xyz="${elbow_roll_joint_init_xyz}" rpy="${elbow_roll_joint_init_rpy}" />
-            <limit lower="-1.8326" upper="1.8326" effort="100.0" velocity="1.0" />
+            <limit lower="-3.8" upper="1.4" effort="100.0" velocity="1.0" />
             <axis xyz="0 0 1" />
         </joint>
@@ -207,5 +207,5 @@
             <child link="elbow_pitch" />
 			<origin xyz="${elbow_pitch_joint_init_xyz}" rpy="${elbow_pitch_joint_init_rpy}" />
-            <limit lower="-1.8326" upper="1.8326" effort="100.0" velocity="1.0" />
+            <limit lower="-3.2" upper="0.8" effort="100.0" velocity="1.0" />
             <axis xyz="1 0 0" />
         </joint>
@@ -249,5 +249,5 @@
             <child link="elbow_yaw" />
 			<origin xyz="${elbow_yaw_joint_init_xyz}" rpy="${elbow_yaw_joint_init_rpy}" />
-            <limit lower="-1.8326" upper="1.8326" effort="100.0" velocity="1.0" />
+            <limit lower="-3.2" upper="0.8" effort="100.0" velocity="1.0" />
             <axis xyz="0 -1 0" />
         </joint>
@@ -289,5 +289,5 @@
             <child link="wrist_pitch" />
 			<origin xyz="${wrist_pitch_joint_init_xyz}" rpy="${wrist_pitch_joint_init_rpy}" />
-            <limit lower="-1.8326" upper="1.8326" effort="100.0" velocity="1.0" />
+            <limit lower="-3.1" upper="0.8" effort="100.0" velocity="1.0" />
             <axis xyz="1 0 0" />
         </joint>
@@ -329,5 +329,5 @@
             <child link="wrist_roll" />
 			<origin xyz="${wrist_roll_joint_init_xyz}" rpy="${wrist_roll_joint_init_rpy}" />
-            <limit lower="-2.61799" upper="2.61799" effort="100.0" velocity="1.0" />
+            <limit lower="-3.8" upper="1.4" effort="100.0" velocity="1.0" />
             <axis xyz="0 0 1" />
         </joint>
